Commit message: added a)low-poly collision meshes b)proper joint limits c)imu link and joint

File: bittle.urdf (robot description, URDF)
Before this commit: robot bittle, 11 links, 10 joints
Links:
- added link imu_link, mass 0.001; visual mesh filename=../meshes/obj/Cube.011.obj scale=1.0 1.0 1.0
- added link mainboard_link, mass 0.001; visual mesh filename=../meshes/obj/Plane.obj scale=1.0 1.0 1.0
- link base-frame-link: mass 0.116 -> 0.108; geometry collision mesh filename=../meshes/obj/base_frame.001.obj scale=1.0 1.0 1.0; visual mesh filename=../meshes/obj/base_frame.obj scale=1.0 1.0 1.0
- link battery-link: geometry collision mesh filename=../meshes/obj/battery.001.obj scale=1.0 1.0 1.0; visual mesh filename=../meshes/obj/battery.obj scale=1.0 1.0 1.0
- link cover-link: geometry collision mesh filename=../meshes/obj/cover.001.obj scale=1.0 1.0 1.0; visual mesh filename=../meshes/obj/cover.obj scale=1.0 1.0 1.0
- link left-back-knee-link: geometry collision mesh filename=../meshes/obj/left_knee.002.obj scale=1.0 1.0 1.0; visual mesh filename=../meshes/obj/left_knee.001.obj scale=1.0 1.0 1.0
- link left-back-shoulder-link: geometry collision mesh filename=../meshes/obj/shoulder.004.obj scale=1.0 1.0 1.0; visual mesh filename=../meshes/obj/shoulder.001.obj scale=1.0 1.0 1.0
- link left-front-knee-link: geometry collision mesh filename=../meshes/obj/left_knee.003.obj scale=1.0 1.0 1.0; visual mesh filename=../meshes/obj/left_knee.obj scale=1.0 1.0 1.0
- link left-front-shoulder-link: geometry collision mesh filename=../meshes/obj/shoulder.007.obj scale=1.0 1.0 1.0; visual mesh filename=../meshes/obj/shoulder.obj scale=1.0 1.0 1.0
- link right-back-knee-link: geometry collision mesh filename=../meshes/obj/right_knee.002.obj scale=1.0 1.0 1.0; visual mesh filename=../meshes/obj/right_knee.001.obj scale=1.0 1.0 1.0
- link right-back-shoulder-link: geometry collision mesh filename=../meshes/obj/shoulder.005.obj scale=1.0 1.0 1.0; visual mesh filename=../meshes/obj/shoulder.002.obj scale=1.0 1.0 1.0
- link right-front-knee-link: geometry collision mesh filename=../meshes/obj/right_knee.003.obj scale=1.0 1.0 1.0; visual mesh filename=../meshes/obj/right_knee.obj scale=1.0 1.0 1.0
- link right-front-shoulder-link: geometry collision mesh filename=../meshes/obj/shoulder.006.obj scale=1.0 1.0 1.0; visual mesh filename=../meshes/obj/shoulder.003.obj scale=1.0 1.0 1.0
Joints:
- added joint imu_joint: type fixed, parent mainboard_link, child imu_link, origin xyz=-0.00652 0.00827 0.00586 rpy=0 0 -3.14159
- added joint mainboard_joint: type fixed, parent base-frame-link, child mainboard_link, origin xyz=0.00652 -0.00827 0.06423 rpy=0 0 0
- joint left-back-knee-joint: limit lower=-1.5708 upper=1.5708 effort=1.0 velocity=1.5708 -> lower=-1.22173 upper=1.48353 effort=1.0 velocity=1.5708
- joint left-back-shoulder-joint: limit lower=-1.5708 upper=1.5708 effort=1.0 velocity=1.5708 -> lower=-1.5708 upper=1.22173 effort=1.0 velocity=1.5708
- joint left-front-knee-joint: limit lower=-1.5708 upper=1.5708 effort=1.0 velocity=1.5708 -> lower=-1.22173 upper=1.48353 effort=1.0 velocity=1.5708
- joint left-front-shoulder-joint: limit lower=-1.5708 upper=1.5708 effort=1.0 velocity=1.5708 -> lower=-1.5708 upper=1.22173 effort=1.0 velocity=1.5708
- joint right-back-knee-joint: limit lower=-1.5708 upper=1.5708 effort=1.0 velocity=1.5708 -> lower=-1.22173 upper=1.48353 effort=1.0 velocity=1.5708
- joint right-back-shoulder-joint: limit lower=-1.5708 upper=1.5708 effort=1.0 velocity=1.5708 -> lower=-1.5708 upper=1.22173 effort=1.0 velocity=1.5708
- joint right-front-knee-joint: limit lower=-1.5708 upper=1.5708 effort=1.0 velocity=1.5708 -> lower=-1.22173 upper=1.48353 effort=1.0 velocity=1.5708
- joint right-front-shoulder-joint: limit lower=-1.5708 upper=1.5708 effort=1.0 velocity=1.5708 -> lower=-1.5708 upper=1.22173 effort=1.0 velocity=1.5708
